Commit message: refactor diffbot hardware interface and update configs

File: diffbot_description/urdf/diffbot.urdf.xacro (robot description, xacro)
@@ -1,23 +1,54 @@
 <?xml version="1.0"?>
 <robot name="diffbot" xmlns:xacro="http://www.ros.org/wiki/xacro">
-  <!-- LINKS -->
-  <link name="base_link"/>
-  <link name="left_wheel"/>
-  <link name="right_wheel"/>
-  <!-- JOINTS -->
+  <!-- ================= PARAMETERS ================= -->
+  <xacro:property name="wheel_radius" value="0.034"/>
+  <xacro:property name="wheel_separation" value="0.264"/>
+  <xacro:property name="wheel_width" value="0.03"/>
+  <xacro:property name="half_wheel_sep" value="${wheel_separation/2.0}"/>
+  <!-- ================= BASE LINK ================= -->
+  <link name="base_link">
+    <visual>
+      <geometry>
+        <box size="0.3 0.2 0.1"/>
+      </geometry>
+      <origin xyz="0 0 0.05"/>
+    </visual>
+  </link>
+  <!-- ================= LEFT WHEEL ================= -->
+  <link name="left_wheel">
+    <visual>
+      <geometry>
+        <cylinder radius="${wheel_radius}" length="${wheel_width}"/>
+      </geometry>
+      <origin xyz="0 0 0" rpy="1.5707 0 0"/>
+    </visual>
+  </link>
   <joint name="left_wheel_joint" type="continuous">
     <parent link="base_link"/>
     <child link="left_wheel"/>
+    <!-- y = + half separation -->
+    <origin xyz="0 ${half_wheel_sep} ${wheel_radius}" rpy="0 0 0"/>
     <axis xyz="0 1 0"/>
   </joint>
+  <!-- ================= RIGHT WHEEL ================= -->
+  <link name="right_wheel">
+    <visual>
+      <geometry>
+        <cylinder radius="${wheel_radius}" length="${wheel_width}"/>
+      </geometry>
+      <origin xyz="0 0 0" rpy="1.5707 0 0"/>
+    </visual>
+  </link>
   <joint name="right_wheel_joint" type="continuous">
     <parent link="base_link"/>
     <child link="right_wheel"/>
+    <!-- y = - half separation -->
+    <origin xyz="0 -${half_wheel_sep} ${wheel_radius}" rpy="0 0 0"/>
     <axis xyz="0 1 0"/>
   </joint>
-  <!-- ROS2 CONTROL -->
+  <!-- ================= ROS2 CONTROL ================= -->
   <ros2_control name="TeensySystem" type="system">
     <hardware>
-      <plugin>diffbot_hardware/TeensyDiffDrive</plugin>
+      <plugin>diffbot_hardware/DiffBotSystemHardware</plugin>
       <param name="serial_port">/dev/ttyACM0</param>
       <param name="baudrate">115200</param>
@@ -34,4 +65,3 @@
     </joint>
   </ros2_control>
-   <!-- <xacro:diffbot_ros2_control/> -->
 </robot>
